Commit message: add all files

File: resources/robots/XBot/urdf/XBot-L.urdf (robot description, URDF)
Before this commit: robot XBot-L, 91 links, 90 joints
Links:
- link base_link: geometry collision box size=0.4 0.4 0.4; visual mesh filename=/data/wanshan/Desktop/robotics/humanoid-gym/resources/robot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
- link left_ankle_pitch_link: geometry visual mesh filename=/data/wanshan/Desktop/robotics/humanoid-gym/resources/robot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
- link left_ankle_pitch_linkage1_link: geometry visual mesh filename=/data/wanshan/Desktop/robotics/humanoid-gym/resources/robot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
- link left_ankle_pitch_linkage2_link: geometry visual mesh filename=/data/wanshan/Desktop/robotics/humanoid-gym/resources/robot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
- link left_ankle_pitch_motor1_link: geometry visual mesh filename=/data/wanshan/Desktop/robotics/humanoid-gym/resources/robot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
- link left_ankle_pitch_motor2_link: geometry visual mesh filename=/data/wanshan/Desktop/robotics/humanoid-gym/resources/robot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
- link left_ankle_roll_link: geometry collision mesh filename=/data/wanshan/Desktop/robotics/humanoid-gym/resources/robot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; visual mesh filename=/data/wanshan/Desktop/robotics/humanoid-gym/resources/robot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
- link left_arm_base_link: geometry collision mesh filename=/data/wanshan/Desktop/robotics/humanoid-gym/resources/robot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; visual mesh filename=/data/wanshan/Desktop/robotics/humanoid-gym/resources/robot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
- link left_arm_yaw_link: geometry collision mesh filename=/data/wanshan/Desktop/robotics/humanoid-gym/resources/robot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; visual mesh filename=/data/wanshan/Desktop/robotics/humanoid-gym/resources/robot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
- link left_elbow_pitch_link: geometry collision mesh filename=/data/wanshan/Desktop/robotics/humanoid-gym/resources/robot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; visual mesh filename=/data/wanshan/Desktop/robotics/humanoid-gym/resources/robot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
- link left_elbow_yaw_link: geometry collision mesh filename=/data/wanshan/Desktop/robotics/humanoid-gym/resources/robot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; visual mesh filename=/data/wanshan/Desktop/robotics/humanoid-gym/resources/robot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
- link left_foot_ee_link: geometry visual mesh filename=/data/wanshan/Desktop/robotics/humanoid-gym/resources/robot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
- link left_hand_ee_link: geometry collision mesh filename=/data/wanshan/Desktop/robotics/humanoid-gym/resources/robot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; visual mesh filename=/data/wanshan/Desktop/robotics/humanoid-gym/resources/robot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
- link left_hand_index_rota_link1: geometry collision mesh filename=/data/wanshan/Desktop/robotics/humanoid-gym/resources/robot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; visual mesh filename=/data/wanshan/Desktop/robotics/humanoid-gym/resources/robot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
- link left_hand_index_rota_link2: geometry collision mesh filename=/data/wanshan/Desktop/robotics/humanoid-gym/resources/robot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; visual mesh filename=/data/wanshan/Desktop/robotics/humanoid-gym/resources/robot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
- link left_hand_index_tip: geometry collision mesh filename=/data/wanshan/Desktop/robotics/humanoid-gym/resources/robot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; visual mesh filename=/data/wanshan/Desktop/robotics/humanoid-gym/resources/robot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
- link left_hand_link: geometry collision mesh filename=/data/wanshan/Desktop/robotics/humanoid-gym/resources/robot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; visual mesh filename=/data/wanshan/Desktop/robotics/humanoid-gym/resources/robot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
- link left_hand_mid_link1: geometry collision mesh filename=/data/wanshan/Desktop/robotics/humanoid-gym/resources/robot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; visual mesh filename=/data/wanshan/Desktop/robotics/humanoid-gym/resources/robot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
- link left_hand_mid_link2: geometry collision mesh filename=/data/wanshan/Desktop/robotics/humanoid-gym/resources/robot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; visual mesh filename=/data/wanshan/Desktop/robotics/humanoid-gym/resources/robot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
- link left_hand_mid_tip: geometry collision mesh filename=/data/wanshan/Desktop/robotics/humanoid-gym/resources/robot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; visual mesh filename=/data/wanshan/Desktop/robotics/humanoid-gym/resources/robot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
- link left_hand_pinky_link1: geometry collision mesh filename=/data/wanshan/Desktop/robotics/humanoid-gym/resources/robot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; visual mesh filename=/data/wanshan/Desktop/robotics/humanoid-gym/resources/robot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
- link left_hand_pinky_link2: geometry collision mesh filename=/data/wanshan/Desktop/robotics/humanoid-gym/resources/robot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; visual mesh filename=/data/wanshan/Desktop/robotics/humanoid-gym/resources/robot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
- link left_hand_pinky_tip: geometry collision mesh filename=/data/wanshan/Desktop/robotics/humanoid-gym/resources/robot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; visual mesh filename=/data/wanshan/Desktop/robotics/humanoid-gym/resources/robot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
- link left_hand_ring_link1: geometry collision mesh filename=/data/wanshan/Desktop/robotics/humanoid-gym/resources/robot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; visual mesh filename=/data/wanshan/Desktop/robotics/humanoid-gym/resources/robot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
- link left_hand_ring_link2: geometry collision mesh filename=/data/wanshan/Desktop/robotics/humanoid-gym/resources/robot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; visual mesh filename=/data/wanshan/Desktop/robotics/humanoid-gym/resources/robot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
- link left_hand_ring_tip: geometry collision mesh filename=/data/wanshan/Desktop/robotics/humanoid-gym/resources/robot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; visual mesh filename=/data/wanshan/Desktop/robotics/humanoid-gym/resources/robot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
- link left_hand_thumb_bend_link: geometry collision mesh filename=/data/wanshan/Desktop/robotics/humanoid-gym/resources/robot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; visual mesh filename=/data/wanshan/Desktop/robotics/humanoid-gym/resources/robot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
- link left_hand_thumb_rota_link1: geometry collision mesh filename=/data/wanshan/Desktop/robotics/humanoid-gym/resources/robot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; visual mesh filename=/data/wanshan/Desktop/robotics/humanoid-gym/resources/robot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
- link left_hand_thumb_rota_link2: geometry collision mesh filename=/data/wanshan/Desktop/robotics/humanoid-gym/resources/robot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; visual mesh filename=/data/wanshan/Desktop/robotics/humanoid-gym/resources/robot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
- link left_hand_thumb_tip: geometry collision mesh filename=/data/wanshan/Desktop/robotics/humanoid-gym/resources/robot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; visual mesh filename=/data/wanshan/Desktop/robotics/humanoid-gym/resources/robot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
- link left_knee_link: geometry collision mesh filename=/data/wanshan/Desktop/robotics/humanoid-gym/resources/robot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; visual mesh filename=/data/wanshan/Desktop/robotics/humanoid-gym/resources/robot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
- link left_knee_linkage_link: geometry visual mesh filename=/data/wanshan/Desktop/robotics/humanoid-gym/resources/robot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
- link left_knee_motor_link: geometry visual mesh filename=/data/wanshan/Desktop/robotics/humanoid-gym/resources/robot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
- link left_leg_pitch_link: geometry collision mesh filename=/data/wanshan/Desktop/robotics/humanoid-gym/resources/robot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; visual mesh filename=/data/wanshan/Desktop/robotics/humanoid-gym/resources/robot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
- link left_leg_roll_link: geometry visual mesh filename=/data/wanshan/Desktop/robotics/humanoid-gym/resources/robot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
- link left_leg_yaw_link: geometry visual mesh filename=/data/wanshan/Desktop/robotics/humanoid-gym/resources/robot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
- link left_shoulder_pitch_link: geometry collision mesh filename=/data/wanshan/Desktop/robotics/humanoid-gym/resources/robot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; visual mesh filename=/data/wanshan/Desktop/robotics/humanoid-gym/resources/robot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
- link left_shoulder_roll_link: geometry collision mesh filename=/data/wanshan/Desktop/robotics/humanoid-gym/resources/robot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; visual mesh filename=/data/wanshan/Desktop/robotics/humanoid-gym/resources/robot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
- link left_wrist_roll_link: geometry collision mesh filename=/data/wanshan/Desktop/robotics/humanoid-gym/resources/robot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; visual mesh filename=/data/wanshan/Desktop/robotics/humanoid-gym/resources/robot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
- link left_wrist_yaw_link: geometry visual mesh filename=/data/wanshan/Desktop/robotics/humanoid-gym/resources/robot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
- link neck_base_link: geometry collision mesh filename=/data/wanshan/Desktop/robotics/humanoid-gym/resources/robot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; visual mesh filename=/data/wanshan/Desktop/robotics/humanoid-gym/resources/robot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
- link neck_pitch_link: geometry collision mesh filename=/data/wanshan/Desktop/robotics/humanoid-gym/resources/robot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; visual mesh filename=/data/wanshan/Desktop/robotics/humanoid-gym/resources/robot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
- link neck_yaw_link: geometry collision mesh filename=/data/wanshan/Desktop/robotics/humanoid-gym/resources/robot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; visual mesh filename=/data/wanshan/Desktop/robotics/humanoid-gym/resources/robot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
- link realsense_link: geometry collision mesh filename=/data/wanshan/Desktop/robotics/humanoid-gym/resources/robot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; visual mesh filename=/data/wanshan/Desktop/robotics/humanoid-gym/resources/robot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
- link right_ankle_pitch_link: geometry visual mesh filename=/data/wanshan/Desktop/robotics/humanoid-gym/resources/robot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
- link right_ankle_pitch_linkage1_link: geometry visual mesh filename=/data/wanshan/Desktop/robotics/humanoid-gym/resources/robot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
- link right_ankle_pitch_linkage2_link: geometry visual mesh filename=/data/wanshan/Desktop/robotics/humanoid-gym/resources/robot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
- link right_ankle_pitch_motor1_link: geometry visual mesh filename=/data/wanshan/Desktop/robotics/humanoid-gym/resources/robot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
- link right_ankle_pitch_motor2_link: geometry visual mesh filename=/data/wanshan/Desktop/robotics/humanoid-gym/resources/robot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
- link right_ankle_roll_link: geometry collision mesh filename=/data/wanshan/Desktop/robotics/humanoid-gym/resources/robot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; visual mesh filename=/data/wanshan/Desktop/robotics/humanoid-gym/resources/robot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
- link right_arm_base_link: geometry collision mesh filename=/data/wanshan/Desktop/robotics/humanoid-gym/resources/robot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; visual mesh filename=/data/wanshan/Desktop/robotics/humanoid-gym/resources/robot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
- link right_arm_yaw_link: geometry collision mesh filename=/data/wanshan/Desktop/robotics/humanoid-gym/resources/robot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; visual mesh filename=/data/wanshan/Desktop/robotics/humanoid-gym/resources/robot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
- link right_elbow_pitch_link: geometry collision mesh filename=/data/wanshan/Desktop/robotics/humanoid-gym/resources/robot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; visual mesh filename=/data/wanshan/Desktop/robotics/humanoid-gym/resources/robot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
- link right_elbow_yaw_link: geometry collision mesh filename=/data/wanshan/Desktop/robotics/humanoid-gym/resources/robot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; visual mesh filename=/data/wanshan/Desktop/robotics/humanoid-gym/resources/robot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
- link right_foot_ee_link: geometry visual mesh filename=/data/wanshan/Desktop/robotics/humanoid-gym/resources/robot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
- link right_hand_ee_link: geometry collision mesh filename=/data/wanshan/Desktop/robotics/humanoid-gym/resources/robot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; visual mesh filename=/data/wanshan/Desktop/robotics/humanoid-gym/resources/robot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
- link right_hand_index_rota_link1: geometry collision mesh filename=/data/wanshan/Desktop/robotics/humanoid-gym/resources/robot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; visual mesh filename=/data/wanshan/Desktop/robotics/humanoid-gym/resources/robot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
- link right_hand_index_rota_link2: geometry collision mesh filename=/data/wanshan/Desktop/robotics/humanoid-gym/resources/robot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; visual mesh filename=/data/wanshan/Desktop/robotics/humanoid-gym/resources/robot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
- link right_hand_index_tip: geometry collision mesh filename=/data/wanshan/Desktop/robotics/humanoid-gym/resources/robot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; visual mesh filename=/data/wanshan/Desktop/robotics/humanoid-gym/resources/robot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
- link right_hand_link: geometry collision mesh filename=/data/wanshan/Desktop/robotics/humanoid-gym/resources/robot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; visual mesh filename=/data/wanshan/Desktop/robotics/humanoid-gym/resources/robot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
- link right_hand_mid_link1: geometry collision mesh filename=/data/wanshan/Desktop/robotics/humanoid-gym/resources/robot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; visual mesh filename=/data/wanshan/Desktop/robotics/humanoid-gym/resources/robot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
- link right_hand_mid_link2: geometry collision mesh filename=/data/wanshan/Desktop/robotics/humanoid-gym/resources/robot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; visual mesh filename=/data/wanshan/Desktop/robotics/humanoid-gym/resources/robot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
- link right_hand_mid_tip: geometry collision mesh filename=/data/wanshan/Desktop/robotics/humanoid-gym/resources/robot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; visual mesh filename=/data/wanshan/Desktop/robotics/humanoid-gym/resources/robot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
- link right_hand_pinky_link1: geometry collision mesh filename=/data/wanshan/Desktop/robotics/humanoid-gym/resources/robot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; visual mesh filename=/data/wanshan/Desktop/robotics/humanoid-gym/resources/robot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
- link right_hand_pinky_link2: geometry collision mesh filename=/data/wanshan/Desktop/robotics/humanoid-gym/resources/robot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; visual mesh filename=/data/wanshan/Desktop/robotics/humanoid-gym/resources/robot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
- link right_hand_pinky_tip: geometry collision mesh filename=/data/wanshan/Desktop/robotics/humanoid-gym/resources/robot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; visual mesh filename=/data/wanshan/Desktop/robotics/humanoid-gym/resources/robot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
- link right_hand_ring_link1: geometry collision mesh filename=/data/wanshan/Desktop/robotics/humanoid-gym/resources/robot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; visual mesh filename=/data/wanshan/Desktop/robotics/humanoid-gym/resources/robot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
- link right_hand_ring_link2: geometry collision mesh filename=/data/wanshan/Desktop/robotics/humanoid-gym/resources/robot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; visual mesh filename=/data/wanshan/Desktop/robotics/humanoid-gym/resources/robot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
- link right_hand_ring_tip: geometry collision mesh filename=/data/wanshan/Desktop/robotics/humanoid-gym/resources/robot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; visual mesh filename=/data/wanshan/Desktop/robotics/humanoid-gym/resources/robot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
- link right_hand_thumb_bend_link: geometry collision mesh filename=/data/wanshan/Desktop/robotics/humanoid-gym/resources/robot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; visual mesh filename=/data/wanshan/Desktop/robotics/humanoid-gym/resources/robot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
- link right_hand_thumb_rota_link1: geometry collision mesh filename=/data/wanshan/Desktop/robotics/humanoid-gym/resources/robot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; visual mesh filename=/data/wanshan/Desktop/robotics/humanoid-gym/resources/robot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
- link right_hand_thumb_rota_link2: geometry collision mesh filename=/data/wanshan/Desktop/robotics/humanoid-gym/resources/robot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; visual mesh filename=/data/wanshan/Desktop/robotics/humanoid-gym/resources/robot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
- link right_hand_thumb_rota_tip: geometry collision mesh filename=/data/wanshan/Desktop/robotics/humanoid-gym/resources/robot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; visual mesh filename=/data/wanshan/Desktop/robotics/humanoid-gym/resources/robot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
- link right_knee_link: geometry collision mesh filename=/data/wanshan/Desktop/robotics/humanoid-gym/resources/robot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; visual mesh filename=/data/wanshan/Desktop/robotics/humanoid-gym/resources/robot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
- link right_knee_linkage_link: geometry visual mesh filename=/data/wanshan/Desktop/robotics/humanoid-gym/resources/robot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
- link right_knee_motor_link: geometry visual mesh filename=/data/wanshan/Desktop/robotics/humanoid-gym/resources/robot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
- link right_leg_pitch_link: geometry collision mesh filename=/data/wanshan/Desktop/robotics/humanoid-gym/resources/robot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; visual mesh filename=/data/wanshan/Desktop/robotics/humanoid-gym/resources/robot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
- link right_leg_roll_link: geometry visual mesh filename=/data/wanshan/Desktop/robotics/humanoid-gym/resources/robot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
- link right_leg_yaw_link: geometry visual mesh filename=/data/wanshan/Desktop/robotics/humanoid-gym/resources/robot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
- link right_shoulder_pitch_link: geometry collision mesh filename=/data/wanshan/Desktop/robotics/humanoid-gym/resources/robot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; visual mesh filename=/data/wanshan/Desktop/robotics/humanoid-gym/resources/robot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
- link right_shoulder_roll_link: geometry collision mesh filename=/data/wanshan/Desktop/robotics/humanoid-gym/resources/robot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; visual mesh filename=/data/wanshan/Desktop/robotics/humanoid-gym/resources/robot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
- link right_wrist_roll_link: geometry collision mesh filename=/data/wanshan/Desktop/robotics/humanoid-gym/resources/robot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; visual mesh filename=/data/wanshan/Desktop/robotics/humanoid-gym/resources/robot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
- link right_wrist_yaw_link: geometry visual mesh filename=/data/wanshan/Desktop/robotics/humanoid-gym/resources/robot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
- link waist_roll_link: geometry visual mesh filename=/data/wanshan/Desktop/robotics/humanoid-gym/resources/robot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
- link waist_yaw_link: geometry visual mesh filename=/data/wanshan/Desktop/robotics/humanoid-gym/resources/robot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
