Commit message: add mujoco xml file

File: resources/robots/i1/mjcf/i1_1101.urdf (robot description, URDF)
Before this commit: robot i1_1101, 23 links, 22 joints
Joints:
- joint l_arm_pitch_joint: limit lower=0 upper=0 effort=0 velocity=0 -> lower=10 upper=10 effort=40 velocity=6
- joint l_shoulder_pitch_joint: limit lower=0 upper=0 effort=0 velocity=0 -> lower=10 upper=10 effort=40 velocity=6
- joint l_shoulder_roll_joint: limit lower=0 upper=0 effort=0 velocity=0 -> lower=10 upper=10 effort=40 velocity=6
- joint l_shoulder_yaw_joint: limit lower=0 upper=0 effort=0 velocity=0 -> lower=10 upper=10 effort=40 velocity=6
- joint leg_l1_joint: limit lower=-0.9 upper=0.7 effort=200 velocity=12 -> lower=-0.9 upper=0.7 effort=150 velocity=12
- joint leg_l2_joint: limit lower=-0.7 upper=0.05 effort=200 velocity=12 -> lower=-0.7 upper=0.05 effort=150 velocity=12
- joint leg_l3_joint: limit lower=-0.8 upper=0.8 effort=0 velocity=0 -> lower=-0.8 upper=0.8 effort=150 velocity=12
- joint leg_l4_joint: limit lower=-0.1 upper=1.8 effort=200 velocity=12 -> lower=-0.1 upper=1.8 effort=150 velocity=12
- joint leg_l5_joint: limit lower=-0.9 upper=0.2 effort=200 velocity=12 -> lower=-0.9 upper=0.2 effort=40 velocity=6
- joint leg_r1_joint: limit lower=-0.9 upper=0.7 effort=200 velocity=12 -> lower=-0.9 upper=0.7 effort=150 velocity=12
- joint leg_r2_joint: limit lower=-0.7 upper=0.05 effort=200 velocity=12 -> lower=-0.7 upper=0.05 effort=150 velocity=12
- joint leg_r3_joint: limit lower=-0.8 upper=0.8 effort=200 velocity=12 -> lower=-0.8 upper=0.8 effort=150 velocity=12
- joint leg_r4_joint: limit lower=-0.1 upper=1.8 effort=200 velocity=12 -> lower=-0.1 upper=1.8 effort=150 velocity=12
- joint leg_r5_joint: limit lower=-0.9 upper=0.2 effort=200 velocity=12 -> lower=-0.9 upper=0.2 effort=40 velocity=6
- joint loin_yaw_joint: limit lower=0 upper=0 effort=0 velocity=0 -> lower=10 upper=10 effort=40 velocity=6
- joint r_arm_pitch_joint: limit lower=0 upper=0 effort=0 velocity=0 -> lower=10 upper=10 effort=40 velocity=6
- joint r_shoulder_pitch_joint: limit lower=0 upper=0 effort=0 velocity=0 -> lower=10 upper=10 effort=40 velocity=6
- joint r_shoulder_roll_joint: limit lower=0 upper=0 effort=0 velocity=0 -> lower=10 upper=10 effort=40 velocity=6
- joint r_shoulder_yaw_joint: limit lower=0 upper=0 effort=0 velocity=0 -> lower=10 upper=10 effort=40 velocity=6
