Commit message: add i1 (including upper body)

File: resources/robots/i1/mjcf/i1_1101_walk_small.urdf (robot description, URDF)
Before this commit: robot i1_1101, 23 links, 22 joints
Links:
- link leg_l3: geometry collision mesh filename=../mjcf_meshes/leg_l3.STL; visual mesh filename=../mjcf_meshes/leg_l3.STL
Joints:
- joint leg_l1_joint: limit lower=-0.7 upper=0.9 effort=14 velocity=4 -> lower=-0.9 upper=0.7 effort=150 velocity=12; origin xyz=0 0.0495999999994021 -0.0620000000004782 rpy=0 -0.35 0 -> xyz=0 0.0495999999994021 -0.0620000000004782 rpy=0 -0.2 0
- joint leg_l2_joint: limit lower=-0.7 upper=0 effort=14 velocity=4 -> lower=-0.7 upper=0 effort=50 velocity=12
- joint leg_l3_joint: limit lower=-0.8 upper=0.8 effort=14 velocity=4 -> lower=-0.8 upper=0.8 effort=150 velocity=12
- joint leg_l4_joint: limit lower=-0.1 upper=1.6 effort=14 velocity=4 -> lower=-0.1 upper=1.6 effort=150 velocity=12; origin xyz=0 0.0271000000001188 -0.117049999999972 rpy=0 0.7 0 -> xyz=0 0.0271000000001188 -0.117049999999972 rpy=0 0.4 0
- joint leg_l5_joint: limit lower=-0.9 upper=0.2 effort=14 velocity=4 -> lower=-0.9 upper=0.2 effort=40 velocity=6; origin xyz=0 -0.00709999999740331 -0.200000000000092 rpy=0 -0.35 0 -> xyz=0 -0.00709999999740331 -0.200000000000092 rpy=0 -0.2 0
- joint leg_r1_joint: limit lower=-0.7 upper=0.9 effort=14 velocity=4 -> lower=-0.9 upper=0.7 effort=150 velocity=12; origin xyz=0 -0.0496000000005979 -0.0619999999995216 rpy=0 -0.35 0 -> xyz=0 -0.0496000000005979 -0.0619999999995216 rpy=0 -0.2 0
- joint leg_r2_joint: limit lower=0 upper=0.7 effort=14 velocity=4 -> lower=-0.7 upper=0 effort=50 velocity=12
- joint leg_r3_joint: limit lower=-0.8 upper=0.8 effort=14 velocity=4 -> lower=-0.8 upper=0.8 effort=150 velocity=12
- joint leg_r4_joint: limit lower=-0.1 upper=1.6 effort=14 velocity=4 -> lower=-0.1 upper=1.6 effort=150 velocity=12; origin xyz=0 -0.0270999999988379 -0.117050000000269 rpy=0 0.7 0 -> xyz=0 -0.0270999999988379 -0.117050000000269 rpy=0 0.4 0
- joint leg_r5_joint: limit lower=-0.9 upper=0.2 effort=14 velocity=4 -> lower=-0.9 upper=0.2 effort=40 velocity=6; origin xyz=0 0.00715000000367917 -0.200000000000334 rpy=0 -0.35 0 -> xyz=0 0.00715000000367917 -0.200000000000334 rpy=0 -0.2 0

File: resources/robots/i1/urdf/i1_1101.urdf (robot description, URDF)
Before this commit: robot i1_1101, 22 links, 21 joints
Links:
- link leg_l2: geometry visual mesh filename=../mjcf_meshes/leg_l2.STL
- link leg_l3: geometry collision mesh filename=../mjcf_meshes/leg_l3.STL; visual mesh filename=../mjcf_meshes/leg_l3.STL
Joints:
- joint l_arm_pitch_joint: limit lower=0 upper=0 effort=0 velocity=0 -> lower=10 upper=10 effort=40 velocity=6
- joint l_shoulder_pitch_joint: limit lower=0 upper=0 effort=0 velocity=0 -> lower=-0.5 upper=0.5 effort=14 velocity=5
- joint l_shoulder_roll_joint: limit lower=0 upper=0 effort=0 velocity=0 -> lower=10 upper=10 effort=40 velocity=6
- joint l_shoulder_yaw_joint: limit lower=0 upper=0 effort=0 velocity=0 -> lower=10 upper=10 effort=40 velocity=6
- joint leg_l1_joint: limit lower=-0.9 upper=0.7 effort=150 velocity=12 -> lower=-0.7 upper=0.9 effort=14 velocity=4
- joint leg_l2_joint: limit lower=-0.7 upper=0.05 effort=150 velocity=12 -> lower=-0.7 upper=0 effort=14 velocity=4
- joint leg_l3_joint: limit lower=-0.8 upper=0.8 effort=150 velocity=12 -> lower=-0.8 upper=0.8 effort=14 velocity=4
- joint leg_l4_joint: limit lower=-0.1 upper=1.8 effort=150 velocity=12 -> lower=-0.1 upper=1.6 effort=14 velocity=4
- joint leg_l5_joint: limit lower=-0.9 upper=0.2 effort=40 velocity=6 -> lower=-0.9 upper=0.2 effort=14 velocity=4
- joint leg_r1_joint: limit lower=-0.9 upper=0.7 effort=150 velocity=12 -> lower=-0.7 upper=0.9 effort=14 velocity=4
- joint leg_r2_joint: limit lower=-0.7 upper=0.05 effort=150 velocity=12 -> lower=0 upper=0.7 effort=14 velocity=4
- joint leg_r3_joint: limit lower=-0.8 upper=0.8 effort=150 velocity=12 -> lower=-0.8 upper=0.8 effort=14 velocity=4
- joint leg_r4_joint: limit lower=-0.1 upper=1.8 effort=150 velocity=12 -> lower=-0.1 upper=1.6 effort=14 velocity=4; origin xyz=0 -0.0270999999988379 -0.117050000000269 rpy=0 .7 0 -> xyz=0 -0.0270999999988379 -0.117050000000269 rpy=0 0.7 0
- joint leg_r5_joint: limit lower=-0.9 upper=0.2 effort=40 velocity=6 -> lower=-0.9 upper=0.2 effort=14 velocity=4
- joint loin_yaw_joint: limit lower=0 upper=0 effort=0 velocity=0 -> lower=10 upper=10 effort=40 velocity=6
- joint r_arm_pitch_joint: limit lower=0 upper=0 effort=0 velocity=0 -> lower=10 upper=10 effort=40 velocity=6
- joint r_shoulder_pitch_joint: limit lower=0 upper=0 effort=0 velocity=0 -> lower=-0.5 upper=0.5 effort=14 velocity=5
- joint r_shoulder_roll_joint: limit lower=0 upper=0 effort=0 velocity=0 -> lower=10 upper=10 effort=40 velocity=6
- joint r_shoulder_yaw_joint: limit lower=0 upper=0 effort=0 velocity=0 -> lower=10 upper=10 effort=40 velocity=6

File: resources/robots/i1/urdf/i1_1101_small_walk.urdf (robot description, URDF)
Before this commit: robot i1_1101, 23 links, 22 joints
Links:
- removed link world
- link leg_l2: geometry visual mesh filename=../mjcf_meshes/leg_l2.STL
- link leg_l3: geometry collision mesh filename=../mjcf_meshes/leg_l3.STL; visual mesh filename=../mjcf_meshes/leg_l3.STL
Joints:
- removed joint floating_base_joint
- joint l_arm_pitch_joint: type revolute -> fixed
- joint l_shoulder_pitch_joint: type revolute -> fixed
- joint l_shoulder_roll_joint: type revolute -> fixed
- joint l_shoulder_yaw_joint: type revolute -> fixed
- joint leg_l1_joint: limit lower=-0.7 upper=0.9 effort=14 velocity=4 -> lower=-0.9 upper=0.7 effort=150 velocity=12; origin xyz=0 0.0495999999994021 -0.0620000000004782 rpy=0 -0.35 0 -> xyz=0 0.0495999999994021 -0.0620000000004782 rpy=0 -0.2 0
- joint leg_l2_joint: limit lower=-0.7 upper=0 effort=14 velocity=4 -> lower=-0.7 upper=0 effort=50 velocity=12
- joint leg_l3_joint: limit lower=-0.8 upper=0.8 effort=14 velocity=4 -> lower=-0.8 upper=0.8 effort=150 velocity=12
- joint leg_l4_joint: limit lower=-0.1 upper=1.6 effort=14 velocity=4 -> lower=-0.1 upper=1.6 effort=150 velocity=12; origin xyz=0 0.0271000000001188 -0.117049999999972 rpy=0 0.7 0 -> xyz=0 0.0271000000001188 -0.117049999999972 rpy=0 0.4 0
- joint leg_l5_joint: limit lower=-0.9 upper=0.2 effort=14 velocity=4 -> lower=-0.9 upper=0.2 effort=40 velocity=6; origin xyz=0 -0.00709999999740331 -0.200000000000092 rpy=0 -0.35 0 -> xyz=0 -0.00709999999740331 -0.200000000000092 rpy=0 -0.2 0
- joint leg_r1_joint: limit lower=-0.7 upper=0.9 effort=14 velocity=4 -> lower=-0.9 upper=0.7 effort=150 velocity=12; origin xyz=0 -0.0496000000005979 -0.0619999999995216 rpy=0 -0.35 0 -> xyz=0 -0.0496000000005979 -0.0619999999995216 rpy=0 -0.2 0
- joint leg_r2_joint: limit lower=0 upper=0.7 effort=14 velocity=4 -> lower=-0.7 upper=0 effort=50 velocity=12
- joint leg_r3_joint: limit lower=-0.8 upper=0.8 effort=14 velocity=4 -> lower=-0.8 upper=0.8 effort=150 velocity=12
- joint leg_r4_joint: limit lower=-0.1 upper=1.6 effort=14 velocity=4 -> lower=-0.1 upper=1.6 effort=150 velocity=12; origin xyz=0 -0.0270999999988379 -0.117050000000269 rpy=0 0.7 0 -> xyz=0 -0.0270999999988379 -0.117050000000269 rpy=0 0.4 0
- joint leg_r5_joint: limit lower=-0.9 upper=0.2 effort=14 velocity=4 -> lower=-0.9 upper=0.2 effort=40 velocity=6; origin xyz=0 0.00715000000367917 -0.200000000000334 rpy=0 -0.35 0 -> xyz=0 0.00715000000367917 -0.200000000000334 rpy=0 -0.2 0
- joint loin_yaw_joint: type revolute -> fixed
- joint r_arm_pitch_joint: type revolute -> fixed
- joint r_shoulder_pitch_joint: type revolute -> fixed
- joint r_shoulder_roll_joint: type revolute -> fixed
- joint r_shoulder_yaw_joint: type revolute -> fixed

File: resources/robots/i1/urdf/i1_1101_stand.urdf (robot description, URDF)
Before this commit: robot i1_1101, 23 links, 22 joints
Links:
- removed link world
- link leg_l3: geometry collision mesh filename=../mjcf_meshes/leg_l3.STL; visual mesh filename=../mjcf_meshes/leg_l3.STL
Joints:
- removed joint floating_base_joint
- joint l_arm_pitch_joint: type revolute -> fixed
- joint l_shoulder_pitch_joint: type revolute -> fixed
- joint l_shoulder_roll_joint: type revolute -> fixed
- joint l_shoulder_yaw_joint: type revolute -> fixed
- joint leg_l1_joint: limit lower=-0.7 upper=0.9 effort=14 velocity=4 -> lower=-0.9 upper=0.7 effort=150 velocity=12; origin xyz=0 0.0495999999994021 -0.0620000000004782 rpy=0 -0.35 0 -> xyz=0 0.0495999999994021 -0.0620000000004782 rpy=0 0 0
- joint leg_l2_joint: limit lower=-0.7 upper=0 effort=14 velocity=4 -> lower=-0.7 upper=0 effort=50 velocity=12
- joint leg_l3_joint: limit lower=-0.8 upper=0.8 effort=14 velocity=4 -> lower=-0.8 upper=0.8 effort=150 velocity=12
- joint leg_l4_joint: limit lower=-0.1 upper=1.6 effort=14 velocity=4 -> lower=-0.1 upper=1.6 effort=150 velocity=12; origin xyz=0 0.0271000000001188 -0.117049999999972 rpy=0 0.7 0 -> xyz=0 0.0271000000001188 -0.117049999999972 rpy=0 0 0
- joint leg_l5_joint: limit lower=-0.9 upper=0.2 effort=14 velocity=4 -> lower=-0.9 upper=0.2 effort=40 velocity=6; origin xyz=0 -0.00709999999740331 -0.200000000000092 rpy=0 -0.35 0 -> xyz=0 -0.00709999999740331 -0.200000000000092 rpy=0 0 0
- joint leg_r1_joint: limit lower=-0.7 upper=0.9 effort=14 velocity=4 -> lower=-0.9 upper=0.7 effort=150 velocity=12; origin xyz=0 -0.0496000000005979 -0.0619999999995216 rpy=0 -0.35 0 -> xyz=0 -0.0496000000005979 -0.0619999999995216 rpy=0 0 0
- joint leg_r2_joint: limit lower=0 upper=0.7 effort=14 velocity=4 -> lower=-0.7 upper=0 effort=50 velocity=12
- joint leg_r3_joint: limit lower=-0.8 upper=0.8 effort=14 velocity=4 -> lower=-0.8 upper=0.8 effort=150 velocity=12
- joint leg_r4_joint: limit lower=-0.1 upper=1.6 effort=14 velocity=4 -> lower=-0.1 upper=1.6 effort=150 velocity=12; origin xyz=0 -0.0270999999988379 -0.117050000000269 rpy=0 0.7 0 -> xyz=0 -0.0270999999988379 -0.117050000000269 rpy=0 0 0
- joint leg_r5_joint: limit lower=-0.9 upper=0.2 effort=14 velocity=4 -> lower=-0.9 upper=0.2 effort=40 velocity=6; origin xyz=0 0.00715000000367917 -0.200000000000334 rpy=0 -0.35 0 -> xyz=0 0.00715000000367917 -0.200000000000334 rpy=0 0 0
- joint loin_yaw_joint: type revolute -> fixed
- joint r_arm_pitch_joint: type revolute -> fixed
- joint r_shoulder_pitch_joint: type revolute -> fixed
- joint r_shoulder_roll_joint: type revolute -> fixed
- joint r_shoulder_yaw_joint: type revolute -> fixed

File: resources/robots/i1/urdf/i1_full_body.urdf (robot description, URDF)
Before this commit: robot i1_1101, 23 links, 22 joints
Links:
- removed link world
- link leg_l2: geometry visual mesh filename=../mjcf_meshes/leg_l2.STL
- link leg_l3: geometry collision mesh filename=../mjcf_meshes/leg_l3.STL; visual mesh filename=../mjcf_meshes/leg_l3.STL
Joints:
- removed joint floating_base_joint
- joint l_arm_pitch_joint: type revolute -> fixed
- joint l_shoulder_pitch_joint: limit lower=10 upper=10 effort=40 velocity=6 -> lower=-0.5 upper=-0.5 effort=6 velocity=3
- joint l_shoulder_roll_joint: type revolute -> fixed
- joint l_shoulder_yaw_joint: type revolute -> fixed
- joint loin_yaw_joint: type revolute -> fixed
- joint r_arm_pitch_joint: type revolute -> fixed
- joint r_shoulder_pitch_joint: limit lower=10 upper=10 effort=40 velocity=6 -> lower=-0.5 upper=0.5 effort=6 velocity=3
- joint r_shoulder_roll_joint: type revolute -> fixed
- joint r_shoulder_yaw_joint: type revolute -> fixed
