Commit message: add full body urdf and mjcf

File: resources/robots/i1/mjcf/i1_full_body.urdf (robot description, URDF)
Before this commit: robot i1_1101, 23 links, 22 joints
Joints:
- joint l_arm_pitch_joint: limit lower=10 upper=10 effort=40 velocity=6 -> lower=10 upper=10 effort=6 velocity=6
- joint l_shoulder_pitch_joint: axis -0.010704 0.99994 0 -> 0 1 0; limit lower=10 upper=10 effort=40 velocity=6 -> lower=-0.5 upper=0.5 effort=6 velocity=3
- joint r_arm_pitch_joint: limit lower=10 upper=10 effort=40 velocity=6 -> lower=10 upper=10 effort=6 velocity=3
- joint r_shoulder_pitch_joint: origin xyz=0.0015211 -0.1421 0.19236 rpy=0 0 0.010704 -> xyz=0.0015211 -0.1421 0.19236 rpy=0 0 0
- joint r_shoulder_roll_joint: limit lower=10 upper=10 effort=40 velocity=6 -> lower=10 upper=10 effort=6 velocity=3
- joint r_shoulder_yaw_joint: limit lower=10 upper=10 effort=40 velocity=6 -> lower=10 upper=10 effort=6 velocity=3

File: resources/robots/i1/urdf/i1_full_body.urdf (robot description, URDF)
Before this commit: robot i1_1101_full_body, 22 links, 21 joints
Links:
- link l_arm_pitch: mass 0.347006 -> 0.347026
- link l_shoulder_roll: mass 0.123182 -> 0.123184
- link l_shoulder_yaw: mass 0.509094 -> 0.50875
Joints:
- joint l_arm_pitch_joint: limit lower=10 upper=10 effort=40 velocity=6 -> lower=-1.5 upper=1.5 effort=6 velocity=3; type fixed -> revolute
- joint l_shoulder_pitch_joint: axis -0.010704 0.99994 0 -> 0 1 0; limit lower=-0.5 upper=-0.5 effort=6 velocity=3 -> lower=-0.5 upper=0.5 effort=4 velocity=3; origin xyz=-0.0015211 0.1421 0.19236 rpy=0 0 0 -> xyz=0.0015211 0.1421 0.19236 rpy=0 -0.15 0
- joint l_shoulder_roll_joint: limit lower=10 upper=10 effort=40 velocity=6 -> lower=-1.5 upper=0 effort=6 velocity=3; type fixed -> revolute
- joint l_shoulder_yaw_joint: limit lower=10 upper=10 effort=40 velocity=6 -> lower=-1.5 upper=1.5 effort=3 velocity=1; type fixed -> revolute
- joint r_arm_pitch_joint: limit lower=10 upper=10 effort=40 velocity=6 -> lower=-1.5 upper=1.5 effort=6 velocity=3; type fixed -> revolute
- joint r_shoulder_pitch_joint: limit lower=-0.5 upper=0.5 effort=6 velocity=3 -> lower=-0.5 upper=0.5 effort=4 velocity=3; origin xyz=0.0015211 -0.1421 0.19236 rpy=0 0 0.010704 -> xyz=0.0015211 -0.1421 0.19236 rpy=0 -0.15 0
- joint r_shoulder_roll_joint: limit lower=10 upper=10 effort=40 velocity=6 -> lower=-1.5 upper=0 effort=3 velocity=1; type fixed -> revolute
- joint r_shoulder_yaw_joint: limit lower=10 upper=10 effort=40 velocity=6 -> lower=-1.5 upper=1.5 effort=6 velocity=3; type fixed -> revolute
