Commit message: add urdf for full body (18dof)

File: resources/robots/i1/mjcf/i1_full_body_18dof.urdf (robot description, URDF)
Before this commit: robot i1_1101_full_body, 22 links, 21 joints
Links:
- added link world
Joints:
- added joint floating_base_joint: type floating, parent world, child base_link
- joint l_arm_pitch_joint: limit lower=-1.5 upper=1.5 effort=14 velocity=4 -> lower=-1.5 upper=1.5 effort=10 velocity=3
- joint l_shoulder_pitch_joint: limit lower=-0.5 upper=0.5 effort=14 velocity=4 -> lower=-0.5 upper=0.5 effort=10 velocity=3; origin xyz=0.0015211 0.1421 0.19236 rpy=0 0 0 -> xyz=0.0015211 0.1421 0.19236 rpy=0 -0.15 0
- joint l_shoulder_roll_joint: limit lower=-1.5 upper=0 effort=154 velocity=4 -> lower=-1.5 upper=0 effort=10 velocity=3
- joint l_shoulder_yaw_joint: limit lower=-1.5 upper=1.5 effort=14 velocity=4 -> lower=-1.5 upper=1.5 effort=10 velocity=3
- joint r_arm_pitch_joint: limit lower=-1.5 upper=1.5 effort=14 velocity=4 -> lower=-1.5 upper=1.5 effort=10 velocity=3
- joint r_shoulder_pitch_joint: limit lower=-0.5 upper=0.5 effort=14 velocity=4 -> lower=-0.5 upper=0.5 effort=10 velocity=3; origin xyz=0.0015211 -0.1421 0.19236 rpy=0 0 0 -> xyz=0.0015211 -0.1421 0.19236 rpy=0 -0.15 0
- joint r_shoulder_roll_joint: limit lower=-1.5 upper=0 effort=14 velocity=4 -> lower=-1.5 upper=0 effort=10 velocity=3
- joint r_shoulder_yaw_joint: limit lower=-1.5 upper=1.5 effort=14 velocity=4 -> lower=-1.5 upper=1.5 effort=10 velocity=3
